Commit message: update standup backflip

File: legged_gym/resources/robots/Yun1/urdf/yun1.urdf (robot description, URDF)
Before this commit: robot yun1, 17 links, 16 joints
Links:
- removed link fl_foot_Link
- removed link fr_foot_Link
- removed link rl_foot_Link
- removed link rr_foot_Link
- link base_link: mass 2.87129405 -> 2.94983380; geometry collision mesh filename=package://V1.1/meshes/base_link.STL; visual mesh filename=package://V1.1/meshes/base_link.STL
- link fl_calf_Link: mass 0.08358392 -> 0.08362378; geometry collision mesh filename=package://V1.1/meshes/fl_calf_Link.STL; visual mesh filename=package://V1.1/meshes/fl_calf_Link.STL
- link fl_hip_Link: mass 0.40036239 -> 0.40515369; geometry collision mesh filename=package://V1.1/meshes/fl_hip_Link.STL; visual mesh filename=package://V1.1/meshes/fl_hip_Link.STL
- link fl_thigh_Link: mass 0.47156059 -> 0.47143546; geometry collision mesh filename=package://V1.1/meshes/fl_thigh_Link.STL; visual mesh filename=package://V1.1/meshes/fl_thigh_Link.STL
- link fr_calf_Link: mass 0.08358392 -> 0.08362378; geometry collision mesh filename=package://V1.1/meshes/fr_calf_Link.STL; visual mesh filename=package://V1.1/meshes/fr_calf_Link.STL
- link fr_hip_Link: mass 0.40021841 -> 0.40515117; geometry collision mesh filename=package://V1.1/meshes/fr_hip_Link.STL; visual mesh filename=package://V1.1/meshes/fr_hip_Link.STL
- link fr_thigh_Link: mass 0.47156059 -> 0.47143546; geometry collision mesh filename=package://V1.1/meshes/fr_thigh_Link.STL; visual mesh filename=package://V1.1/meshes/fr_thigh_Link.STL
- link rl_calf_Link: mass 0.08358392 -> 0.08362378; geometry collision mesh filename=package://V1.1/meshes/rl_calf_Link.STL; visual mesh filename=package://V1.1/meshes/rl_calf_Link.STL
- link rl_hip_Link: mass 0.40021841 -> 0.40515117; geometry collision mesh filename=package://V1.1/meshes/rl_hip_Link.STL; visual mesh filename=package://V1.1/meshes/rl_hip_Link.STL
- link rl_thigh_Link: mass 0.47156059 -> 0.47143546; geometry collision mesh filename=package://V1.1/meshes/rl_thigh_Link.STL; visual mesh filename=package://V1.1/meshes/rl_thigh_Link.STL
- link rr_calf_Link: mass 0.08358392 -> 0.08362378; geometry collision mesh filename=package://V1.1/meshes/rr_calf_Link.STL; visual mesh filename=package://V1.1/meshes/rr_calf_Link.STL
- link rr_hip_Link: mass 0.40036239 -> 0.40515369; geometry collision mesh filename=package://V1.1/meshes/rr_hip_Link.STL; visual mesh filename=package://V1.1/meshes/rr_hip_Link.STL
- link rr_thigh_Link: mass 0.47156059 -> 0.47143546; geometry collision mesh filename=package://V1.1/meshes/rr_thigh_Link.STL; visual mesh filename=package://V1.1/meshes/rr_thigh_Link.STL
Joints:
- removed joint fl_foot_Joint
- removed joint fr_foot_Joint
- removed joint rl_foot_Joint
- removed joint rr_foot_Joint
